File: SoundSwarm-eagle/soundthings.brd (EAGLE design)
At the start: 100 x 44 mm, 33 parts, among them Q2 IRLB8721PBF

Commit message: Fixed: DC-DC on VDD (switched)
Connections:
- net VBAT: no longer U$7.VIN+
- net VDD: now also U$7.VIN+
Routing:
- net VDD: track 29.8 -> 89.9 mm
- net VBAT: track 102.0 -> 43.8 mm
- net GND: track 221.2 -> 224.6 mm
Changed lines of the file:
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@@
 <wire x1="66.3448" y1="31.496" x2="66.427" y2="31.54" width="0.4064" layer="1"/>
 <wire x1="58.7248" y1="29.6672" x2="58.65" y2="29.57" width="0.4064" layer="1"/>
-<wire x1="80.9752" y1="37.592" x2="83.7184" y2="37.592" width="0.4064" layer="1"/>
-<wire x1="75.0824" y1="31.6992" x2="80.9752" y2="37.592" width="0.4064" layer="1"/>
-<wire x1="66.548" y1="31.6992" x2="75.0824" y2="31.6992" width="0.4064" layer="1"/>
-<wire x1="83.7184" y1="37.592" x2="83.8" y2="37.6" width="0.4064" layer="1"/>
+<wire x1="80.9752" y1="37.6936" x2="83.7184" y2="37.6936" width="0.4064" layer="1"/>
+<wire x1="77.3176" y1="41.3512" x2="80.9752" y2="37.6936" width="0.4064" layer="1"/>
+<wire x1="73.5584" y1="41.3512" x2="77.3176" y2="41.3512" width="0.4064" layer="1"/>
+<wire x1="69.2912" y1="37.084" x2="73.5584" y2="41.3512" width="0.4064" layer="1"/>
+<wire x1="69.2912" y1="34.4424" x2="69.2912" y2="37.084" width="0.4064" layer="1"/>
+<wire x1="66.548" y1="31.6992" x2="69.2912" y2="34.4424" width="0.4064" layer="1"/>
+<wire x1="83.7184" y1="37.6936" x2="83.8" y2="37.6" width="0.4064" layer="1"/>
 <wire x1="66.548" y1="31.6992" x2="66.427" y2="31.54" width="0.4064" layer="1"/>
 <wire x1="91.3384" y1="14.3256" x2="91.3384" y2="15.8496" width="0.4064" layer="1"/>
@@
 <wire x1="49.276" y1="19.5072" x2="49.2" y2="19.54" width="0.4064" layer="1"/>
 <wire x1="49.3776" y1="12.2936" x2="49.4512" y2="12.2606" width="0.4064" layer="1"/>
-<wire x1="46.1264" y1="9.2456" x2="36.2712" y2="9.2456" width="0.4064" layer="1"/>
-<wire x1="49.1744" y1="12.2936" x2="46.1264" y2="9.2456" width="0.4064" layer="1"/>
-<wire x1="36.2712" y1="9.2456" x2="36.2" y2="9.15" width="0.4064" layer="1"/>
-<wire x1="49.1744" y1="12.2936" x2="49.4512" y2="12.2606" width="0.4064" layer="1"/>
-<wire x1="54.1528" y1="7.62" x2="62.1792" y2="7.62" width="0.4064" layer="1"/>
-<wire x1="49.5808" y1="12.192" x2="54.1528" y2="7.62" width="0.4064" layer="1"/>
-<wire x1="62.1792" y1="7.62" x2="62.25" y2="7.6" width="0.4064" layer="1"/>
-<wire x1="49.5808" y1="12.192" x2="49.4512" y2="12.2606" width="0.4064" layer="1"/>
+<wire x1="46.4312" y1="9.2456" x2="37.8968" y2="9.2456" width="0.4064" layer="16"/>
+<wire x1="37.8968" y1="9.2456" x2="36.2712" y2="9.2456" width="0.4064" layer="16"/>
+<wire x1="49.3776" y1="12.192" x2="46.4312" y2="9.2456" width="0.4064" layer="16"/>
+<wire x1="36.2712" y1="9.2456" x2="36.2" y2="9.15" width="0.4064" layer="16"/>
+<wire x1="49.3776" y1="12.192" x2="49.4512" y2="12.2606" width="0.4064" layer="16"/>
+<wire x1="54.1528" y1="7.62" x2="62.1792" y2="7.62" width="0.4064" layer="16"/>
+<wire x1="49.5808" y1="12.192" x2="54.1528" y2="7.62" width="0.4064" layer="16"/>
+<wire x1="62.1792" y1="7.62" x2="62.25" y2="7.6" width="0.4064" layer="16"/>
+<wire x1="49.5808" y1="12.192" x2="49.4512" y2="12.2606" width="0.4064" layer="16"/>
 <wire x1="81.0768" y1="6.8072" x2="83.6168" y2="6.8072" width="0.4064" layer="1"/>
 <wire x1="77.3176" y1="3.048" x2="81.0768" y2="6.8072" width="0.4064" layer="1"/>
-<wire x1="66.8528" y1="3.048" x2="77.3176" y2="3.048" width="0.4064" layer="1"/>
-<wire x1="62.3824" y1="7.5184" x2="66.8528" y2="3.048" width="0.4064" layer="1"/>
+<wire x1="66.7512" y1="3.048" x2="77.3176" y2="3.048" width="0.4064" layer="1"/>
+<wire x1="62.2808" y1="7.5184" x2="66.7512" y2="3.048" width="0.4064" layer="1"/>
 <wire x1="83.6168" y1="6.8072" x2="83.8" y2="6.8" width="0.4064" layer="1"/>
-<wire x1="62.3824" y1="7.5184" x2="62.25" y2="7.6" width="0.4064" layer="1"/>
+<wire x1="62.2808" y1="7.5184" x2="62.25" y2="7.6" width="0.4064" layer="1"/>
 <wire x1="58.6232" y1="28.956" x2="58.6232" y2="29.3624" width="0.4064" layer="16"/>
 <wire x1="49.4792" y1="19.812" x2="58.6232" y2="28.956" width="0.4064" layer="16"/>
-<wire x1="49.4792" y1="12.2936" x2="49.4792" y2="19.812" width="0.4064" layer="16"/>
+<wire x1="49.4792" y1="12.3952" x2="49.4792" y2="19.812" width="0.4064" layer="16"/>
 <wire x1="58.6232" y1="29.3624" x2="58.65" y2="29.57" width="0.4064" layer="16"/>
-<wire x1="49.4792" y1="12.2936" x2="49.4512" y2="12.2606" width="0.4064" layer="16"/>
+<wire x1="49.4792" y1="12.3952" x2="49.4512" y2="12.2606" width="0.4064" layer="16"/>
 <wire x1="30.1752" y1="15.5448" x2="27.432" y2="15.5448" width="0.4064" layer="16"/>
 <wire x1="32.8168" y1="12.9032" x2="30.1752" y2="15.5448" width="0.4064" layer="16"/>
 <wire x1="37.1856" y1="12.9032" x2="32.8168" y2="12.9032" width="0.4064" layer="16"/>
 <wire x1="37.8968" y1="12.192" x2="37.1856" y2="12.9032" width="0.4064" layer="16"/>
-<wire x1="37.8968" y1="10.0584" x2="37.8968" y2="12.192" width="0.4064" layer="16"/>
-<wire x1="37.084" y1="9.2456" x2="37.8968" y2="10.0584" width="0.4064" layer="16"/>
-<wire x1="36.2712" y1="9.2456" x2="37.084" y2="9.2456" width="0.4064" layer="16"/>
+<wire x1="37.8968" y1="9.2456" x2="37.8968" y2="12.192" width="0.4064" layer="16"/>
 <wire x1="27.432" y1="15.5448" x2="27.4" y2="15.62" width="0.4064" layer="16"/>
-<wire x1="36.2712" y1="9.2456" x2="36.2" y2="9.15" width="0.4064" layer="16"/>
 </signal>
 <signal name="SOL-" class="2">
@@
 <contactref element="C3" pad="1"/>
 <contactref element="R11" pad="P$2"/>
-<contactref element="U$7" pad="VIN+"/>
 <wire x1="23.6728" y1="9.144" x2="24.4856" y2="9.144" width="0.4064" layer="1"/>
 <wire x1="22.2504" y1="10.5664" x2="23.6728" y2="9.144" width="0.4064" layer="1"/>
@@
 <wire x1="16.9672" y1="10.668" x2="16.99" y2="10.6" width="0.4064" layer="16"/>
 <wire x1="13.5128" y1="26.2128" x2="13.6699" y2="26.27" width="0.4064" layer="16"/>
-<wire x1="69.596" y1="37.6936" x2="75.3872" y2="37.6936" width="0.4064" layer="1"/>
-<wire x1="67.8688" y1="39.4208" x2="69.596" y2="37.6936" width="0.4064" layer="1"/>
-<wire x1="54.864" y1="39.4208" x2="67.8688" y2="39.4208" width="0.4064" layer="1"/>
-<wire x1="50.1904" y1="34.7472" x2="54.864" y2="39.4208" width="0.4064" layer="1"/>
-<wire x1="32.2072" y1="34.7472" x2="50.1904" y2="34.7472" width="0.4064" layer="1"/>
-<wire x1="31.9024" y1="35.052" x2="32.2072" y2="34.7472" width="0.4064" layer="1"/>
-<wire x1="31.9024" y1="35.2552" x2="31.9024" y2="35.052" width="0.4064" layer="1"/>
-<wire x1="30.988" y1="36.1696" x2="31.9024" y2="35.2552" width="0.4064" layer="1"/>
-<wire x1="27.8384" y1="36.1696" x2="30.988" y2="36.1696" width="0.4064" layer="1"/>
-<wire x1="22.86" y1="31.1912" x2="27.8384" y2="36.1696" width="0.4064" layer="1"/>
-<wire x1="75.3872" y1="37.6936" x2="75.4" y2="37.6" width="0.4064" layer="1"/>
-<wire x1="22.86" y1="31.1912" x2="22.81" y2="31.14" width="0.4064" layer="1"/>
 </signal>
 <signal name="GPIO16">
@@
 <contactref element="U$5" pad="3"/>
 <contactref element="L1" pad="3"/>
+<contactref element="U$7" pad="VIN+"/>
 <wire x1="14.4272" y1="19.5072" x2="14.4272" y2="18.9992" width="0.2032" layer="16"/>
 <wire x1="14.8336" y1="19.9136" x2="14.4272" y2="19.5072" width="0.2032" layer="16"/>
@@
 <wire x1="21.9456" y1="10.4648" x2="36.1696" y2="10.4648" width="0.2032" layer="16"/>
 <wire x1="36.1696" y1="10.4648" x2="36.2" y2="10.45" width="0.2032" layer="16"/>
+<wire x1="75.3872" y1="21.1328" x2="75.3872" y2="37.592" width="0.2032" layer="1"/>
+<wire x1="64.7192" y1="10.4648" x2="75.3872" y2="21.1328" width="0.2032" layer="1"/>
+<wire x1="36.2712" y1="10.4648" x2="64.7192" y2="10.4648" width="0.2032" layer="1"/>
+<wire x1="75.3872" y1="37.592" x2="75.4" y2="37.6" width="0.2032" layer="1"/>
+<wire x1="36.2712" y1="10.4648" x2="36.2" y2="10.45" width="0.2032" layer="1"/>
 </signal>
 <signal name="SCL">

Commit message: SSv2c with fixed VDD battery measurement
Connections:
- net VBAT: no longer R11.P$2
- net VDD: now also R11.P$2
Routing:
- net VDD: track 89.9 -> 114.0 mm
- net VBAT: track 43.8 -> 36.5 mm
Other:
- board text added: "SSv2c LiL MiP MaP"
- board text removed: "SSv2 LiL MiP MaP"
Changed lines of the file:
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@@
 <wire x1="10" y1="28" x2="0" y2="28" width="0" layer="20"/>
 <wire x1="0" y1="28" x2="0" y2="16" width="0" layer="20"/>
-<text x="56.07" y="13.4" size="1.778" layer="25" font="vector" align="center">SSv2
+<text x="56.07" y="13.4" size="1.778" layer="25" font="vector" align="center">SSv2c
 LiL
 MiP
@@
 <contactref element="U$2" pad="3"/>
 <contactref element="C3" pad="1"/>
-<contactref element="R11" pad="P$2"/>
+<wire x1="13.716" y1="29.6672" x2="13.716" y2="26.3144" width="0.4064" layer="16"/>
+<wire x1="16.1544" y1="32.1056" x2="13.716" y2="29.6672" width="0.4064" layer="16"/>
+<wire x1="13.716" y1="26.3144" x2="13.6699" y2="26.27" width="0.4064" layer="16"/>
+<wire x1="16.1544" y1="32.1056" x2="16.17" y2="32.14" width="0.4064" layer="16"/>
 <wire x1="23.6728" y1="9.144" x2="24.4856" y2="9.144" width="0.4064" layer="1"/>
 <wire x1="22.2504" y1="10.5664" x2="23.6728" y2="9.144" width="0.4064" layer="1"/>
@@
 <wire x1="24.4856" y1="9.144" x2="24.51" y2="9.08" width="0.4064" layer="1"/>
 <wire x1="17.0688" y1="10.5664" x2="16.99" y2="10.6" width="0.4064" layer="1"/>
-<wire x1="13.716" y1="29.6672" x2="13.716" y2="26.3144" width="0.4064" layer="16"/>
-<wire x1="16.1544" y1="32.1056" x2="13.716" y2="29.6672" width="0.4064" layer="16"/>
-<wire x1="13.716" y1="26.3144" x2="13.6699" y2="26.27" width="0.4064" layer="16"/>
-<wire x1="16.1544" y1="32.1056" x2="16.17" y2="32.14" width="0.4064" layer="16"/>
-<wire x1="19.6088" y1="31.0896" x2="22.7584" y2="31.0896" width="0.4064" layer="16"/>
-<wire x1="19.304" y1="30.7848" x2="19.6088" y2="31.0896" width="0.4064" layer="16"/>
-<wire x1="17.6784" y1="30.7848" x2="19.304" y2="30.7848" width="0.4064" layer="16"/>
-<wire x1="16.3576" y1="32.1056" x2="17.6784" y2="30.7848" width="0.4064" layer="16"/>
-<wire x1="22.7584" y1="31.0896" x2="22.81" y2="31.14" width="0.4064" layer="16"/>
-<wire x1="16.3576" y1="32.1056" x2="16.17" y2="32.14" width="0.4064" layer="16"/>
-<wire x1="16.9672" y1="11.5824" x2="16.9672" y2="10.668" width="0.4064" layer="16"/>
-<wire x1="10.0584" y1="18.4912" x2="16.9672" y2="11.5824" width="0.4064" layer="16"/>
-<wire x1="10.0584" y1="25.0952" x2="10.0584" y2="18.4912" width="0.4064" layer="16"/>
-<wire x1="11.176" y1="26.2128" x2="10.0584" y2="25.0952" width="0.4064" layer="16"/>
-<wire x1="13.5128" y1="26.2128" x2="11.176" y2="26.2128" width="0.4064" layer="16"/>
+<wire x1="11.176" y1="26.2128" x2="13.5128" y2="26.2128" width="0.4064" layer="16"/>
+<wire x1="10.0584" y1="25.0952" x2="11.176" y2="26.2128" width="0.4064" layer="16"/>
+<wire x1="10.0584" y1="17.5768" x2="10.0584" y2="25.0952" width="0.4064" layer="16"/>
+<wire x1="16.9672" y1="10.668" x2="10.0584" y2="17.5768" width="0.4064" layer="16"/>
+<wire x1="13.5128" y1="26.2128" x2="13.6699" y2="26.27" width="0.4064" layer="16"/>
 <wire x1="16.9672" y1="10.668" x2="16.99" y2="10.6" width="0.4064" layer="16"/>
-<wire x1="13.5128" y1="26.2128" x2="13.6699" y2="26.27" width="0.4064" layer="16"/>
 </signal>
 <signal name="GPIO16">
@@
 <contactref element="L1" pad="3"/>
 <contactref element="U$7" pad="VIN+"/>
+<contactref element="R11" pad="P$2"/>
 <wire x1="14.4272" y1="19.5072" x2="14.4272" y2="18.9992" width="0.2032" layer="16"/>
 <wire x1="14.8336" y1="19.9136" x2="14.4272" y2="19.5072" width="0.2032" layer="16"/>
@@
 <wire x1="16.3576" y1="18.8976" x2="16.32" y2="18.95" width="0.2032" layer="16"/>
 <wire x1="21.9456" y1="9.144" x2="22.01" y2="9.08" width="0.2032" layer="16"/>
-<wire x1="21.9456" y1="10.4648" x2="36.1696" y2="10.4648" width="0.2032" layer="16"/>
+<wire x1="21.9456" y1="10.4648" x2="26.1112" y2="10.4648" width="0.2032" layer="16"/>
+<wire x1="26.1112" y1="10.4648" x2="36.1696" y2="10.4648" width="0.2032" layer="16"/>
 <wire x1="36.1696" y1="10.4648" x2="36.2" y2="10.45" width="0.2032" layer="16"/>
+<wire x1="22.86" y1="30.3784" x2="22.86" y2="31.0896" width="0.2032" layer="16"/>
+<wire x1="28.6512" y1="24.5872" x2="22.86" y2="30.3784" width="0.2032" layer="16"/>
+<wire x1="28.6512" y1="18.6944" x2="28.6512" y2="24.5872" width="0.2032" layer="16"/>
+<wire x1="26.1112" y1="16.1544" x2="28.6512" y2="18.6944" width="0.2032" layer="16"/>
+<wire x1="26.1112" y1="10.4648" x2="26.1112" y2="16.1544" width="0.2032" layer="16"/>
+<wire x1="22.86" y1="31.0896" x2="22.81" y2="31.14" width="0.2032" layer="16"/>
 <wire x1="75.3872" y1="21.1328" x2="75.3872" y2="37.592" width="0.2032" layer="1"/>
 <wire x1="64.7192" y1="10.4648" x2="75.3872" y2="21.1328" width="0.2032" layer="1"/>
